File: buttons.kicad_pcb (KiCad board)
At the start: 2 copper layers, 30.7 x 35.3 mm, 16 parts, among them J1 Conn_01x02, J3 Conn_01x11, SW1 SW_SPST, SW2 SW_SPST, U1 TLC555xP, U2 74LS14

Commit message: revision 2.0
Parts:
- J3: value Conn_01x11 -> Conn_01x10; footprint Connector_PinHeader_2.54mm:PinHeader_1x11_P2.54mm_Vertical -> Connector_PinHeader_2.54mm:PinHeader_1x10_P2.54mm_Vertical
- R1, R2: value 22k -> 10k
- R3, R4: value 100k -> 1k
- moved C5 14.4 mm to (83.0, 59.2)
- moved C1 4.60 mm to (69.9, 64.5), turned to 180 degrees
- moved C2 3.45 mm to (69.9, 59.9), turned to 180 degrees
- moved J3 2.55 mm to (71.1, 45.7)
- moved C4 0.51 mm to (95.2, 59.2)
- moved SW1 0.13 mm to (77.6, 69.9)
Connections:
- J3 pad 10: /thr -> /clk
- J3 pad 8: /~{sw} -> /dis
- J3 pad 9: /dis -> /thr
- R1 pad 1: Net-(C1-Pad1) -> Net-(R1-Pad1)
- R1 pad 2: Net-(R1-Pad2) -> Net-(C1-Pad1)
- R2 pad 1: Net-(C2-Pad1) -> Net-(R2-Pad1)
- R2 pad 2: Net-(R2-Pad2) -> Net-(C2-Pad1)
- R3 pad 2: Net-(C1-Pad1) -> Net-(R1-Pad1)
- R4 pad 2: Net-(C2-Pad1) -> Net-(R2-Pad1)
- SW1 pad 2: Net-(R1-Pad2) -> Net-(R1-Pad1)
- SW2 pad 2: Net-(R2-Pad2) -> Net-(R2-Pad1)
- SW_MAN1 pad 3: /~{sw} -> Net-(SW_MAN1-Pad3)
- U2 pad 1: Net-(R1-Pad2) -> Net-(C1-Pad1)
- U2 pad 3: Net-(R2-Pad2) -> Net-(C2-Pad1)
- U2 pad 5: /~{sw} -> Net-(SW_MAN1-Pad3)
- U2 pad 8: /~{sw} -> Net-(SW_MAN1-Pad3)
Routing:
- net Net-(R2-Pad2): track 29.4 -> 0.00 mm
- net /~{sw}: track 26.5 -> 0.00 mm
- net Net-(R2-Pad1): track 0.00 -> 24.5 mm
- net Net-(R1-Pad2): track 24.4 -> 0.00 mm
- net Net-(SW_MAN1-Pad3): track 0.00 -> 22.2 mm
- net Net-(R1-Pad1): track 0.00 -> 19.8 mm
- net /b1: track 13.9 -> 16.4 mm
- net Net-(C2-Pad1): track 15.1 -> 13.1 mm
- net /b: track 4.96 -> 3.17 mm
- net Net-(C1-Pad1): track 14.8 -> 16.4 mm
- net /sw: track 14.7 -> 15.8 mm
- net /b2: track 12.9 -> 13.9 mm
- net /~{b}: track 4.22 -> 3.17 mm
- net /~{a}: track 4.22 -> 3.17 mm
- net /a: track 4.22 -> 3.17 mm
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Other:
- board size 30.7 x 35.3 mm -> 30.7 x 34.9 mm
- board text added: "GND"
- board text added: "Knoepfchen 2.0"
- board text added: "VCC"
- board text removed: "~s"
