File: buttons.kicad_sch (KiCad schematic)
At the start: 16 parts, among them J1 Conn_01x02, J3 Conn_01x11, SW1 SW_SPST, SW2 SW_SPST, U1 TLC555xP, U2 74LS14

Commit message: removed old comment
Parts:
- C4: value (none) -> 10nF
Other:
- note added: "Power connector for breadboard"
- note removed: "Connect a resistor R from 10(clk) to 11(thr) and a capacitor C from 10 to GND. Leave 9 NC. clk will have 50% duty cycle and a frequency of 1/(2ln(2)RC) For example: C=470nF R=1eX f=1,531,914.89e-X"
- note removed: "Two power connectors for the breadboard power rail. It is sufficient to connect only one."
Changed lines of the file:
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@@
     (effects (font (size 1.27 1.27)) (justify left bottom))
   )
-  (text "Two power connectors\nfor the breadboard \npower rail. It is\nsufficient to connect\nonly one."
-    (at 17.78 87.63 0)
+  (text "Power connector\nfor breadboard" (at 17.78 87.63 0)
     (effects (font (size 1.27 1.27)) (justify left bottom))
   )
@@
   (text "These are spare negaters. \nPull input to Vcc/GND if not used."
     (at 226.06 48.26 0)
-    (effects (font (size 1.27 1.27)) (justify left bottom))
-  )
-  (text "Connect a resistor R\nfrom 10(clk) to 11(thr) \nand a capacitor C from \n10 to GND. Leave 9 NC.\n\nclk will have 50% \nduty cycle and a \nfrequency of \n1/(2ln(2)RC)\n\nFor example:\nC=470nF\nR=1eX\nf=1,531,914.89e-X"
-    (at 260.35 139.7 0)
     (effects (font (size 1.27 1.27)) (justify left bottom))
   )
@@
       (effects (font (size 1.27 1.27)) (justify left))
     )
-    (property "Value" "" (id 1) (at 52.07 126.9999 0)
+    (property "Value" "10nF" (id 1) (at 52.07 126.9999 0)
       (effects (font (size 1.27 1.27)) (justify left))
     )

Commit message: changed cap value to match pcb
Parts:
- C4: value 10nF -> (none)
Changed lines of the file:
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@@
       (effects (font (size 1.27 1.27)) (justify left))
     )
-    (property "Value" "10nF" (id 1) (at 52.07 126.9999 0)
+    (property "Value" "" (id 1) (at 52.07 126.9999 0)
       (effects (font (size 1.27 1.27)) (justify left))
     )
@@
     )
     (path "/06a5a61e-cc48-49eb-a313-c00bf1c3412c"
-      (reference "C4") (unit 1) (value "10nF") (footprint "Capacitor_THT:C_Disc_D5.0mm_W2.5mm_P5.00mm")
+      (reference "C4") (unit 1) (value "100nF") (footprint "Capacitor_THT:C_Disc_D5.0mm_W2.5mm_P5.00mm")
     )
     (path "/ec499889-f4fa-4ddb-bcc0-8d1eed5d901d"

Commit message: revision 2.0
Parts:
- removed J3: Conn_01x11, Connector_PinHeader_2.54mm:PinHeader_1x11_P2.54mm_Vertical, symbol Connector_Generic:Conn_01x11
- added J3: (no value), symbol Connector_Generic:Conn_01x10
- C4: value (none) -> 100nF
- R1, R2: value 22k -> 10k
- R3, R4: value 100k -> 1k
Connections:
- net a: now also J3.3 (Pin_3)
- net b: now also J3.1 (Pin_1)
- net b1: now also J3.5 (Pin_5)
- net b2: now also J3.6 (Pin_6)
- net clk: now also J3.10 (Pin_10)
- net dis: now also J3.8 (Pin_8)
- net sw: now also J3.7 (Pin_7)
- net thr: now also J3.9 (Pin_9)
- net ~{a}: now also J3.4 (Pin_4)
- net ~{b}: now also J3.2 (Pin_2)
- net at R2.1, R4.2: now also SW2.2 (B); no longer C2.1
- net at R2.2, U2.3: now also C2.1; no longer SW2.2 (B)
- net at R1.2, U2.1: now also C1.1; no longer SW1.2 (B)
- net at R1.1, R3.2: now also SW1.2 (B); no longer C1.1
- net ~{sw}: no longer names the net of SW_MAN1.3 (C), U2.5, U2.8
Other:
- moved on the sheet: C1, C2, C4, C5, J1, R1, R2, R3, R4, R5, SW1, SW2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
